File: motor-controller-pcb/motor-controller-pcb.kicad_pcb (KiCad board)
At the start: 2 copper layers, 90 x 65 mm, 15 parts, among them J1 Conn_01x06_Pin, J2 Conn_01x06_Pin, J3 Conn_01x06_Pin, J4 Conn_01x06_Pin, J5 Conn_01x04_Pin, J6 Conn_01x04_Pin, M1 Conn_01x02_Pin, M2 Conn_01x02_Pin, M3 Conn_01x02_Pin, M4 Conn_01x02_Pin

Commit message: feat: pcb
Parts:
- added J7: Conn_01x08_Pin, Connector_PinHeader_2.54mm:PinHeader_1x08_P2.54mm_Vertical, F.Cu at (145.0, 115.0)
Connections:
- A1 pad 1: unconnected-(A1-GPIO0-Pad1) -> /GP0
- A1 pad 14: unconnected-(A1-GPIO10-Pad14)_1 -> /GP10
- A1 pad 16: unconnected-(A1-GPIO12-Pad16)_1 -> /GP12
- A1 pad 19: unconnected-(A1-GPIO14-Pad19) -> /GP14
- A1 pad 2: unconnected-(A1-GPIO1-Pad2)_1 -> /GP1
- A1 pad 20: unconnected-(A1-GPIO15-Pad20) -> /GP15
- A1 pad 21: unconnected-(A1-GPIO16-Pad21)_1 -> /GP16
- A1 pad 22: unconnected-(A1-GPIO17-Pad22) -> /GP17
Routing:
- net /GP1: track 0.00 -> 81.4 mm
- net /GP0: track 0.00 -> 67.3 mm
- net +5V: track 164.3 -> 123.2 mm
- net /GP12: track 0.00 -> 35.9 mm
- net /GP10: track 0.00 -> 26.4 mm
- net /GP14: track 0.00 -> 21.3 mm
- net /GP15: track 0.00 -> 18.3 mm
- net /GP17: track 0.00 -> 13.0 mm
- net /GP16: track 0.00 -> 9.29 mm
Other:
- board text added: "Robocup 2025 SBHS PCB by Hamzah Ahmed"
