File: motor-controller-pcb/motor-controller-pcb.kicad_sch (KiCad schematic)
At the start: 11 parts, among them J1 Conn_01x06_Pin, J2 Conn_01x06_Pin, J3 Conn_01x06_Pin, J4 Conn_01x06_Pin, J5 Conn_01x04_Pin, J6 Conn_01x04_Pin, M1 Conn_01x02_Pin, M2 Conn_01x02_Pin, M3 Conn_01x02_Pin, M4 Conn_01x02_Pin

Commit message: feat: pcb
Parts:
- added J7: Conn_01x08_Pin, Connector_PinHeader_2.54mm:PinHeader_1x08_P2.54mm_Vertical, symbol Connector:Conn_01x08_Pin
Connections:
- net GP0: now reaches A1.1 (GPIO0)
- net GP0: now also J7.1 (Pin_1)
- net GP10: now reaches A1.14 (GPIO10)
- net GP10: now also J7.3 (Pin_3)
- net GP12: now reaches A1.16 (GPIO12)
- net GP12: now also J7.4 (Pin_4)
- net GP14: now reaches A1.19 (GPIO14)
- net GP14: now also J7.5 (Pin_5)
- net GP1: now reaches A1.2 (GPIO1)
- net GP1: now also J7.2 (Pin_2)
- net GP15: now reaches A1.20 (GPIO15)
- net GP15: now also J7.6 (Pin_6)
- net GP16: now reaches A1.21 (GPIO16)
- net GP16: now also J7.7 (Pin_7)
- net GP17: now reaches A1.22 (GPIO17)
- net GP17: now also J7.8 (Pin_8)
- no-connect marks 24 -> 16
Changed lines of the file:
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@@
-	)
-	(no_connect
-		(at 157.48 72.39)
-	)
-	(no_connect
-		(at 157.48 97.79)
-	)
-	(no_connect
-		(at 157.48 110.49)
-	)
-	(no_connect
-		(at 157.48 107.95)
 	)
 	(no_connect
@@
 	)
 	(no_connect
-		(at 157.48 102.87)
-	)
-	(no_connect
-		(at 203.2 74.93)
-	)
-	(no_connect
 		(at 185.42 49.53)
 	)
@@
 	)
 	(no_connect
-		(at 203.2 77.47)
-	)
-	(no_connect
 		(at 203.2 100.33)
 	)
@@
 	(no_connect
 		(at 85.09 80.01)
-	)
-	(no_connect
-		(at 157.48 74.93)
 	)
 	(wire
@@
 		)
 	)
+	(label "GP1"
+		(at 83.82 45.72 0)
+		(effects
+			(font
+				(size 1.27 1.27)
+			)
+			(justify left bottom)
+		)
+	)
+	(label "GP17"
+		(at 83.82 60.96 0)
+		(effects
+			(font
+				(size 1.27 1.27)
+			)
+			(justify left bottom)
+		)
+	)
+	(label "GP15"
+		(at 83.82 55.88 0)
+		(effects
+			(font
+				(size 1.27 1.27)
+			)
+			(justify left bottom)
+		)
+	)
 	(label "Encoder 2"
 		(at 203.2 82.55 0)
@@
 		)
 	)
+	(label "GP12"
+		(at 83.82 50.8 0)
+		(effects
+			(font
+				(size 1.27 1.27)
+			)
+			(justify left bottom)
+		)
+	)
 	(label "Encoder 1"
 		(at 157.48 100.33 180)
@@
 		)
 	)
+	(label "GP15"
+		(at 157.48 110.49 180)
+		(effects
+			(font
+				(size 1.27 1.27)
+			)
+			(justify right bottom)
+		)
+	)
+	(label "GP16"
+		(at 83.82 58.42 0)
+		(effects
+			(font
+				(size 1.27 1.27)
+			)
+			(justify left bottom)
+		)
+	)
+	(label "GP0"
+		(at 83.82 43.18 0)
+		(effects
+			(font
+				(size 1.27 1.27)
+			)
+			(justify left bottom)
+		)
+	)
+	(label "GP10"
+		(at 83.82 48.26 0)
+		(effects
+			(font
+				(size 1.27 1.27)
+			)
+			(justify left bottom)
+		)
+	)
+	(label "GP16"
+		(at 203.2 74.93 0)
+		(effects
+			(font
+				(size 1.27 1.27)
+			)
+			(justify left bottom)
+		)
+	)
 	(label "Encoder 4"
 		(at 203.2 87.63 0)
@@
 		)
 	)
+	(label "GP14"
+		(at 157.48 107.95 180)
+		(effects
+			(font
+				(size 1.27 1.27)
+			)
+			(justify right bottom)
+		)
+	)
 	(label "Encoder 3"
 		(at 157.48 105.41 180)
@@
 		)
 	)
+	(label "GP14"
+		(at 83.82 53.34 0)
+		(effects
+			(font
+				(size 1.27 1.27)
+			)
+			(justify left bottom)
+		)
+	)
+	(label "GP0"
+		(at 157.48 72.39 180)
+		(effects
+			(font
+				(size 1.27 1.27)
+			)
+			(justify right bottom)
+		)
+	)
 	(label "Encoder 1"
 		(at 97.79 77.47 0)
@@
 		)
 	)
+	(label "GP10"
+		(at 157.48 97.79 180)
+		(effects
+			(font
+				(size 1.27 1.27)
+			)
+			(justify right bottom)
+		)
+	)
+	(label "GP1"
+		(at 157.48 74.93 180)
+		(effects
+			(font
+				(size 1.27 1.27)
+			)
+			(justify right bottom)
+		)
+	)
+	(label "GP17"
+		(at 203.2 77.47 0)
+		(effects
+			(font
+				(size 1.27 1.27)
+			)
+			(justify left bottom)
+		)
+	)
 	(label "Encoder 3"
 		(at 97.79 118.11 0)
@@
 			)
 			(justify left bottom)
+		)
+	)
+	(label "GP12"
+		(at 157.48 102.87 180)
+		(effects
+			(font
+				(size 1.27 1.27)
+			)
+			(justify right bottom)
 		)
 	)
@@
 	)
 	(symbol
+		(lib_id "Connector:Conn_01x08_Pin")
+		(at 78.74 50.8 0)
+		(unit 1)
+		(exclude_from_sim no)
+		(in_bom yes)
+		(on_board yes)
+		(dnp no)
+		(fields_autoplaced yes)
+		(property "Reference" "J7"
+			(at 79.375 38.1 0)
+			(effects
+				(font
+					(size 1.27 1.27)
+				)
+			)
+		)
+		(property "Value" "Conn_01x08_Pin"
+			(at 79.375 40.64 0)
+			(effects
+				(font
+					(size 1.27 1.27)
+				)
+			)
+		)
+		(property "Footprint" "Connector_PinHeader_2.54mm:PinHeader_1x08_P2.54mm_Vertical"
+			(at 78.74 50.8 0)
+			(effects
+				(font
+					(size 1.27 1.27)
+				)
+				(hide yes)
+			)
+		)
+		(property "Datasheet" "~"
+			(at 78.74 50.8 0)
+			(effects
+				(font
+					(size 1.27 1.27)
+				)
+				(hide yes)
+			)
+		)
+		(property "Description" "Generic connector, single row, 01x08, script generated"
+			(at 78.74 50.8 0)
+			(effects
+				(font
+					(size 1.27 1.27)
+				)
+				(hide yes)
+			)
+		)
+		(pin "8"
+		)
+		(pin "3"
+		)
+		(pin "5"
+		)
+		(pin "6"
+		)
+		(pin "4"
+		)
+		(pin "7"
+		)
+		(pin "2"
+		)
+		(pin "1"
+		)
+		(instances
+			(project ""
+				(path "/521a5f8e-be65-4be3-9b63-a6be4ecbc76a"
+					(reference "J7")
+					(unit 1)
+				)
+			)
+		)
+	)
+	(symbol
 		(lib_id "Connector:Conn_01x04_Pin")
 		(at 152.4 90.17 0)
@@
 		(dnp no)
 		(property "Reference" "J6"
-			(at 153.035 82.55 0)
+			(at 142.748 88.138 0)
 			(effects
 				(font
@@
 		)
 		(property "Value" "Conn_01x04_Pin"
-			(at 153.035 85.09 0)
+			(at 140.462 89.916 0)
 			(effects
 				(font
@@
 		(on_board yes)
 		(dnp no)
-		(fields_autoplaced yes)
 		(property "Reference" "J5"
-			(at 153.035 72.39 0)
+			(at 143.002 82.042 0)
 			(effects
 				(font
@@
 		)
 		(property "Value" "Conn_01x04_Pin"
-			(at 153.035 74.93 0)
-			(effects
-				(font
+			(at 142.748 80.01 0)
+			(effects
+				(font
